Commit message: arm finally working sorta

File: src/arm/arm_description/urdf/sliding_arm.urdf.xacro (robot description, xacro)
@@ -4,6 +4,16 @@
   <material name="grey"><color rgba="0.5 0.5 0.5 1"/></material>
   <link name="world"/>
+  <link name="base_link">
+    <inertial>
+      <mass value="0.1"/>
+      <inertia ixx="0.0001" ixy="0" ixz="0" iyy="0.0001" iyz="0" izz="0.0001"/>
+    </inertial>
+  </link>
+  <joint name="world_fixed" type="fixed">
+    <parent link="world"/>
+    <child link="base_link"/>
+  </joint>
   <joint name="base_sliding_joint" type="prismatic">
-    <parent link="world"/>
+    <parent link="base_link"/>
     <child link="slider_link"/>
     <origin xyz="0 0 0.05" rpy="0 0 0"/>

Commit message: added new urdf viewer package for testing joint movements

File: src/arm/arm_description/urdf/sliding_arm.urdf.xacro (robot description, xacro)
@@ -39,5 +39,5 @@
     <child link="arm_link_1"/>
     <origin xyz="0 0 0.05" rpy="0 0 0"/>
-    <axis xyz="0 0 1"/>
+    <axis xyz="0 1 0"/>
     <limit effort="100" lower="-3.14" upper="3.14" velocity="1.0"/>
   </joint>
