Commit message: working arm urdf with correct dof sync, just need to add joint limits

File: src/arm/urdf_viewer/urdf/robot.urdf (robot description, URDF)
Before this commit: robot arm_model_1, 16 links, 15 joints
Joints:
- joint closing_elbow_loop_1_frame: origin xyz=0.354444 0.308505 -0.001 rpy=2.20082e-15 -2.1689e-16 2.28701 -> xyz=0.305568 0.356979 -0.001 rpy=1.60818e-15 -3.83372e-16 2.43364
- joint closing_elbow_loop_1_z_frame: origin xyz=0.354444 0.308505 0.099 rpy=2.20082e-15 -2.1689e-16 2.28701 -> xyz=0.305568 0.356979 0.099 rpy=1.60818e-15 -3.83372e-16 2.43364
- joint closing_elbow_loop_2_frame: origin xyz=-0.0862161 -0.0750419 5.55112e-17 rpy=-3.14159 -1.44343e-16 -2.42538 -> xyz=-0.0743273 -0.0868328 5.55112e-17 rpy=3.14159 2.33498e-17 -2.27875
- joint closing_elbow_loop_2_z_frame: origin xyz=-0.0862161 -0.0750419 -0.1 rpy=-3.14159 -1.44343e-16 -2.42538 -> xyz=-0.0743273 -0.0868328 -0.1 rpy=3.14159 2.33498e-17 -2.27875
- joint closing_shoulder_loop_1_frame: origin xyz=-0.105291 -0.0444783 -0.001 rpy=4.73085e-16 -2.41288e-15 -1.1711 -> xyz=-0.0977981 -0.059161 -0.001 rpy=4.73045e-16 -2.16216e-15 -1.02676
- joint closing_shoulder_loop_1_z_frame: origin xyz=-0.105291 -0.0444783 0.099 rpy=4.73085e-16 -2.41288e-15 -1.1711 -> xyz=-0.0977981 -0.059161 0.099 rpy=4.73045e-16 -2.16216e-15 -1.02676
- joint closing_shoulder_loop_2_frame: origin xyz=9.71445e-17 0.4699 -0.03275 rpy=-4.37096e-16 6.39738e-33 -1.5708 -> xyz=1.38778e-16 0.4699 -0.03275 rpy=-4.37096e-16 -4.05289e-32 -1.5708
- joint closing_shoulder_loop_2_z_frame: origin xyz=1.52656e-16 0.4699 0.06725 rpy=-4.37096e-16 6.39738e-33 -1.5708 -> xyz=1.94289e-16 0.4699 0.06725 rpy=-4.37096e-16 -4.05289e-32 -1.5708
- joint elbow_1: origin xyz=-7.28584e-17 1.11022e-16 -0.03275 rpy=4.73085e-16 -2.41288e-15 -1.1711 -> xyz=3.22225e-16 3.33067e-16 -0.03275 rpy=4.73045e-16 -2.16216e-15 -1.02676
- joint elbow_2: mimic (none) -> joint=elbow_1 multiplier=1.0; origin xyz=-0.105291 -0.0444783 -0.03275 rpy=4.73085e-16 -2.41288e-15 -1.1711 -> xyz=-0.0977981 -0.059161 -0.03275 rpy=4.73045e-16 -2.16216e-15 -1.02676
- joint elbow_end_1: mimic (none) -> joint=elbow_1 multiplier=1.0; origin xyz=0.354444 0.308505 -0.001 rpy=-3.14159 -1.22729e-15 2.28701 -> xyz=0.305568 0.356979 -0.001 rpy=-3.14159 -1.37615e-15 2.43364
- joint shoulder_1: origin xyz=-0.015875 0.01905 0.048625 rpy=1.82266e-16 3.51114e-16 -1.1711 -> xyz=-0.015875 0.01905 0.048625 rpy=1.90309e-16 2.77821e-16 -1.02676
- joint shoulder_2: mimic (none) -> joint=shoulder_1 multiplier=-1.0; origin xyz=-0.015875 0.13335 0.016875 rpy=-3.14159 7.88209e-16 -1.1711 -> xyz=-0.015875 0.13335 0.016875 rpy=-3.14159 7.57238e-16 -1.02676
- joint shoulder_end_1: mimic (none) -> joint=shoulder_1 multiplier=1.0; origin xyz=-5.37764e-17 -0.4699 0 rpy=3.14159 -3.56188e-33 -1.72312e-17 -> xyz=-8.32667e-17 -0.4699 0 rpy=-3.14159 -2.90661e-32 2.70029e-17
- joint slider: limit lower=-0.226078 upper=0.0239215 effort=10 velocity=10 -> lower=-0.25 upper=1.66533e-16 effort=10 velocity=10; origin xyz=-0.08599 0.0510785 0.0762 rpy=-1.5708 6.62236e-16 -2.49816e-16 -> xyz=0.0762 0.075 0.08599 rpy=-1.5708 1.5708 0

Commit message: made script more complete, updated readme

File: src/arm/urdf_viewer/urdf/robot.urdf (robot description, URDF)
Before this commit: robot urdf, 16 links, 15 joints
Joints:
- joint closing_elbow_loop_1_frame: origin xyz=0.305568 0.356979 -0.001 rpy=1.60818e-15 -3.83372e-16 2.43364 -> xyz=0.385056 0.269328 -0.001 rpy=1.90482e-15 2.27584e-16 2.18115
- joint closing_elbow_loop_1_z_frame: origin xyz=0.305568 0.356979 0.099 rpy=1.60818e-15 -3.83372e-16 2.43364 -> xyz=0.385056 0.269328 0.099 rpy=1.90482e-15 2.27584e-16 2.18115
- joint closing_elbow_loop_2_frame: origin xyz=-0.0743273 -0.0868328 5.55112e-17 rpy=3.14159 2.33498e-17 -2.27875 -> xyz=-0.0936623 -0.0655123 -2.77556e-17 rpy=3.14159 -1.02144e-17 -2.53123
- joint closing_elbow_loop_2_z_frame: origin xyz=-0.0743273 -0.0868328 -0.1 rpy=3.14159 2.33498e-17 -2.27875 -> xyz=-0.0936623 -0.0655123 -0.1 rpy=3.14159 -1.02144e-17 -2.53123
- joint closing_shoulder_loop_1_frame: origin xyz=-0.0977981 -0.059161 -0.001 rpy=4.73045e-16 -2.16216e-15 -1.02676 -> xyz=-0.0975658 -0.0595432 -0.001 rpy=3.51171e-16 -2.14865e-15 -1.02285
- joint closing_shoulder_loop_1_z_frame: origin xyz=-0.0977981 -0.059161 0.099 rpy=4.73045e-16 -2.16216e-15 -1.02676 -> xyz=-0.0975658 -0.0595432 0.099 rpy=3.51171e-16 -2.14865e-15 -1.02285
- joint closing_shoulder_loop_2_frame: origin xyz=1.38778e-16 0.4699 -0.03275 rpy=-4.37096e-16 -4.05289e-32 -1.5708 -> xyz=6.93889e-17 0.4699 -0.03275 rpy=-4.37096e-16 8.74776e-32 -1.5708
- joint closing_shoulder_loop_2_z_frame: origin xyz=1.94289e-16 0.4699 0.06725 rpy=-4.37096e-16 -4.05289e-32 -1.5708 -> xyz=1.249e-16 0.4699 0.06725 rpy=-4.37096e-16 8.74776e-32 -1.5708
- joint elbow_1: origin xyz=3.22225e-16 3.33067e-16 -0.03275 rpy=4.73045e-16 -2.16216e-15 -1.02676 -> xyz=-7.89299e-17 2.22045e-16 -0.03275 rpy=3.51171e-16 -2.14865e-15 -1.02285
- joint elbow_2: origin xyz=-0.0977981 -0.059161 -0.03275 rpy=4.73045e-16 -2.16216e-15 -1.02676 -> xyz=-0.0975658 -0.0595432 -0.03275 rpy=3.51171e-16 -2.14865e-15 -1.02285
- joint elbow_end_1: origin xyz=0.305568 0.356979 -0.001 rpy=-3.14159 -1.37615e-15 2.43364 -> xyz=0.385056 0.269328 -0.001 rpy=-3.14159 -9.37689e-16 2.18115
- joint shoulder_1: origin xyz=-0.015875 0.01905 0.048625 rpy=1.90309e-16 2.77821e-16 -1.02676 -> xyz=-0.015875 0.01905 0.048625 rpy=2.28672e-16 3.18144e-16 -1.02285
- joint shoulder_2: origin xyz=-0.015875 0.13335 0.016875 rpy=-3.14159 7.57238e-16 -1.02676 -> xyz=-0.015875 0.13335 0.016875 rpy=-3.14159 7.55239e-16 -1.02285
- joint shoulder_end_1: origin xyz=-8.32667e-17 -0.4699 0 rpy=-3.14159 -2.90661e-32 2.70029e-17 -> xyz=-1.50054e-16 -0.4699 0 rpy=-3.14159 -7.17803e-32 -1.28001e-17
- joint slider: limit lower=-0.25 upper=1.66533e-16 effort=10 velocity=10 -> lower=-0.25 upper=7.79956e-09 effort=10 velocity=10
