Commit message: gazebo robot driving

File: src/navigation/rover_description/urdf/robot.urdf (robot description, URDF)
Before this commit: robot roverbody_urdf, 12 links, 11 joints
Joints:
- joint wheel_1: axis 0 0 1 -> 0 0 -1
- joint wheel_2: axis 0 0 1 -> 0 0 -1
- joint wheel_3: axis 0 0 1 -> 0 0 -1

File: src/navigation/roverbody_urdf/robot copy.urdf (robot description, URDF)
Before this commit: robot roverbody_urdf, 12 links, 11 joints
Links:
- link bearing_block: mass 1.28596 -> 1e-09
- link front_plate: mass 12.8268 -> 1e-09; geometry collision mesh filename=package://assets/corner_bracket_8020.stl; collision mesh filename=package://assets/corner_bracket_8020.stl
- link part1: mass 1.26312 -> 1e-09
- link part_1: mass 1.44032 -> 1e-09
- link part_1_3: mass 1.44032 -> 1e-09
- link part_1_4: mass 1.44032 -> 1e-09
- link part_1_5: mass 1.44032 -> 1e-09
- link part_1_6: mass 1.44032 -> 1e-09
- link part_1_7: mass 1.44032 -> 1e-09
- link part_4: mass 1.19385 -> 1e-09
- link part_5: mass 1.26312 -> 1e-09
- link part_9: mass 1.28596 -> 1e-09
Joints:
- joint main_l: origin xyz=0.239856 0.469254 -0.0801256 rpy=-1.5708 -1.37096e-16 3.14159 -> xyz=0.239856 0.47631 -0.0801256 rpy=1.5708 -0.0664034 -1.11022e-16
- joint sub2_l: origin xyz=0.113405 -0.0060173 -1.30048e-09 rpy=3.14159 -2.86425e-26 -0.0530108 -> xyz=0.113176 -0.00937701 -1.30048e-09 rpy=3.14159 3.48009e-24 -0.0826644
- joint sub2_r: origin xyz=1.11022e-16 8.32667e-17 -0.56 rpy=6.78906e-26 -4.2799e-26 0.0437451 -> xyz=-3.33067e-16 0 -0.56 rpy=7.62338e-24 1.14871e-23 0.0369093
- joint sub_l: origin xyz=-0.239014 0.0881738 -0.0269688 rpy=6.34714e-27 2.37928e-26 -3.08898 -> xyz=0.234047 -0.10062 -0.0199132 rpy=8.59465e-31 3.27328e-31 -7.81868e-16
- joint wheel_1: origin xyz=0.285421 0.261127 -0.0270556 rpy=-1.14868e-17 1.33339e-16 2.44389 -> xyz=-0.298757 -0.245757 -0.02 rpy=-1.14868e-17 1.33339e-16 -0.816718
- joint wheel_2: origin xyz=-0.187242 -0.135406 -0.0170868 rpy=2.45551e-16 -1.76174e-16 -0.868424 -> xyz=-0.191174 -0.129795 -0.0170868 rpy=2.45551e-16 -1.76174e-16 -0.898078
- joint wheel_3: origin xyz=0.175762 -0.154667 -0.0170868 rpy=2.61297e-16 -3.92524e-17 0.702372 -> xyz=0.171099 -0.159811 -0.0170868 rpy=2.61297e-16 -3.92524e-17 0.672719
- joint wheel_6: origin xyz=0.299229 -0.245183 -0.0270556 rpy=8.10526e-17 7.58707e-17 -2.32318 -> xyz=0.296572 -0.248391 -0.0270556 rpy=8.02313e-17 7.67391e-17 -2.33395
