Commit message: moved rover model into separate folder and fixed rigid body

File: src/navigation/rover_gazebo/urdf/rover_gazebo.urdf.xacro (robot description, xacro)
@@ -20,5 +20,5 @@
       <plugin>gz_ros2_control/GazeboSimSystem</plugin>
     </hardware>
-    <joint name="wheel_1">
+    <joint name="jwheel_l1">
       <command_interface name="velocity">
         <param name="min">-10</param>
@@ -28,5 +28,5 @@
       <state_interface name="velocity"/>
     </joint>
-    <joint name="wheel_2">
+    <joint name="jwheel_l2">
       <command_interface name="velocity">
         <param name="min">-10</param>
@@ -36,5 +36,5 @@
       <state_interface name="velocity"/>
     </joint>
-    <joint name="wheel_3">
+    <joint name="jwheel_l3">
       <command_interface name="velocity">
         <param name="min">-10</param>
@@ -44,5 +44,5 @@
       <state_interface name="velocity"/>
     </joint>
-    <joint name="wheel_4">
+    <joint name="jwheel_r3">
       <command_interface name="velocity">
         <param name="min">-10</param>
@@ -52,5 +52,5 @@
       <state_interface name="velocity"/>
     </joint>
-    <joint name="wheel_5">
+    <joint name="jwheel_r2">
       <command_interface name="velocity">
         <param name="min">-10</param>
@@ -60,5 +60,5 @@
       <state_interface name="velocity"/>
     </joint>
-    <joint name="wheel_6">
+    <joint name="jwheel_r1">
       <command_interface name="velocity">
         <param name="min">-10</param>
