Commit message: added end effector control

File: src/arm/arm_gazebo/urdf/arm_gazebo.urdf.xacro (robot description, xacro)
@@ -16,4 +16,6 @@
       - shoulder_1   (revolute)
       - elbow_1      (revolute)
+      - wrist        (revolute)
+      - claw         (revolute)
     Mimic joints (velocity derived from primary via multiplier):
       - shoulder_2     mirrors shoulder_1, multiplier: -1.0
@@ -47,4 +49,20 @@
         <param name="min">-0.67</param>
         <param name="max">0.67</param>
+      </command_interface>
+      <state_interface name="position"/>
+      <state_interface name="velocity"/>
+    </joint>
+    <joint name="wrist">
+      <command_interface name="velocity">
+        <param name="min">-1.0</param>
+        <param name="max">1.0</param>
+      </command_interface>
+      <state_interface name="position"/>
+      <state_interface name="velocity"/>
+    </joint>
+    <joint name="claw">
+      <command_interface name="velocity">
+        <param name="min">-0.5</param>
+        <param name="max">0.5</param>
       </command_interface>
       <state_interface name="position"/>
@@ -107,3 +125,9 @@
     <implicitSpringDamper>1</implicitSpringDamper>
   </gazebo>
+  <gazebo reference="wrist">
+    <implicitSpringDamper>1</implicitSpringDamper>
+  </gazebo>
+  <gazebo reference="claw">
+    <implicitSpringDamper>1</implicitSpringDamper>
+  </gazebo>
 </robot>

File: src/arm/urdf_viewer/urdf/robot.urdf (robot description, URDF)
Before this commit: robot urdf, 16 links, 15 joints
Links:
- added link part_1, mass 1e-09; collision mesh filename=package://urdf_viewer/urdf/assets/part_1.stl; collision mesh filename=package://urdf_viewer/urdf/assets/part_1__2.stl
- added link part_1_2, mass 1e-09; collision mesh filename=package://urdf_viewer/urdf/assets/part_1__3.stl; collision mesh filename=package://urdf_viewer/urdf/assets/part_1__4.stl
- link 6inch_shorter_arm_body_3: geometry collision mesh filename=package://urdf_viewer/urdf/assets/6inch_shorter_arm_body.stl; collision mesh filename=package://urdf_viewer/urdf/assets/part_1.stl
Joints:
- added joint claw: type revolute, parent part_1, child part_1_2, origin xyz=-0.0212 0.03175 -0.0197 rpy=1.5708 1.5708 0, axis 0 0 1, limit lower=-0.785398 upper=0.279253 effort=10 velocity=10
- added joint wrist: type revolute, parent 6inch_shorter_arm_body_3, child part_1, origin xyz=-0.0517585 0.033841 -0.016875 rpy=-1.5708 -0.0628288 -2.26574, axis 0 0 1, limit lower=-3.141592653589793 upper=3.141592653589793 effort=10 velocity=10
- joint closing_elbow_loop_1_frame: origin xyz=0.385056 0.269328 -0.001 rpy=1.90482e-15 2.27584e-16 2.18115 -> xyz=0.300895 0.360927 -0.001 rpy=1.66184e-15 -1.42637e-15 2.44665
- joint closing_elbow_loop_1_z_frame: origin xyz=0.385056 0.269328 0.099 rpy=1.90482e-15 2.27584e-16 2.18115 -> xyz=0.300895 0.360927 0.099 rpy=1.66184e-15 -1.42637e-15 2.44665
- joint closing_elbow_loop_2_frame: origin xyz=-0.0936623 -0.0655123 -2.77556e-17 rpy=3.14159 -1.02144e-17 -2.53123 -> xyz=-0.0731907 -0.087793 -2.77556e-17 rpy=3.14159 5.09899e-18 -2.26574
- joint closing_elbow_loop_2_z_frame: origin xyz=-0.0936623 -0.0655123 -0.1 rpy=3.14159 -1.02144e-17 -2.53123 -> xyz=-0.0731907 -0.087793 -0.1 rpy=3.14159 5.09899e-18 -2.26574
- joint closing_shoulder_loop_1_frame: origin xyz=-0.0975658 -0.0595432 -0.001 rpy=3.51171e-16 -2.14865e-15 -1.02285 -> xyz=-0.0927271 -0.0668295 -0.001 rpy=8.48745e-18 -1.90415e-15 -0.946305
- joint closing_shoulder_loop_1_z_frame: origin xyz=-0.0975658 -0.0595432 0.099 rpy=3.51171e-16 -2.14865e-15 -1.02285 -> xyz=-0.0927271 -0.0668295 0.099 rpy=8.48745e-18 -1.90415e-15 -0.946305
- joint closing_shoulder_loop_2_frame: origin xyz=6.93889e-17 0.4699 -0.03275 rpy=-4.37096e-16 8.74776e-32 -1.5708 -> xyz=1.11022e-16 0.4699 -0.03275 rpy=-4.37096e-16 -4.13476e-32 -1.5708
- joint closing_shoulder_loop_2_z_frame: origin xyz=1.249e-16 0.4699 0.06725 rpy=-4.37096e-16 8.74776e-32 -1.5708 -> xyz=1.38778e-16 0.4699 0.06725 rpy=-4.37096e-16 -4.13476e-32 -1.5708
- joint elbow_1: origin xyz=-7.89299e-17 2.22045e-16 -0.03275 rpy=3.51171e-16 -2.14865e-15 -1.02285 -> xyz=-5.47305e-15 0 -0.03275 rpy=8.48745e-18 -1.90415e-15 -0.946305
- joint elbow_2: origin xyz=-0.0975658 -0.0595432 -0.03275 rpy=3.51171e-16 -2.14865e-15 -1.02285 -> xyz=-0.0927271 -0.0668295 -0.03275 rpy=8.48745e-18 -1.90415e-15 -0.946305
- joint elbow_end_1: origin xyz=0.385056 0.269328 -0.001 rpy=-3.14159 -9.37689e-16 2.18115 -> xyz=0.300895 0.360927 -0.001 rpy=-3.14159 -1.39355e-15 2.44665
- joint shoulder_1: origin xyz=-0.015875 0.01905 0.048625 rpy=2.28672e-16 3.18144e-16 -1.02285 -> xyz=-0.015875 0.01905 0.048625 rpy=2.55946e-16 3.01651e-16 -0.946305
- joint shoulder_2: origin xyz=-0.015875 0.13335 0.016875 rpy=-3.14159 7.55239e-16 -1.02285 -> xyz=-0.015875 0.13335 0.016875 rpy=-3.14159 3.01651e-16 -0.946305
- joint shoulder_end_1: origin xyz=-1.50054e-16 -0.4699 0 rpy=-3.14159 -7.17803e-32 -1.28001e-17 -> xyz=-1.17961e-16 -0.4699 -1.38778e-17 rpy=3.14159 8.03022e-33 -5.89544e-17
- joint slider: limit lower=-0.25 upper=7.79956e-09 effort=10 velocity=10 -> lower=-0.205617 upper=0.0443825 effort=10 velocity=10; origin xyz=0.0762 0.075 0.08599 rpy=-1.5708 1.5708 0 -> xyz=0.0762 0.0306175 0.08599 rpy=-1.5708 1.5708 0

Commit message: improved urdf inertia and stuff for arm

File: src/arm/arm_gazebo/urdf/arm_gazebo.urdf.xacro (robot description, xacro)
@@ -131,3 +131,20 @@
     <implicitSpringDamper>1</implicitSpringDamper>
   </gazebo>
+  <!-- High friction + contact stiffness on claw fingers so objects don't phase through -->
+  <gazebo reference="part_1">
+    <mu1>1.5</mu1>
+    <mu2>1.5</mu2>
+    <kp>1e6</kp>
+    <kd>100</kd>
+    <minDepth>0.001</minDepth>
+    <maxVel>0.1</maxVel>
+  </gazebo>
+  <gazebo reference="part_1_2">
+    <mu1>1.5</mu1>
+    <mu2>1.5</mu2>
+    <kp>1e6</kp>
+    <kd>100</kd>
+    <minDepth>0.001</minDepth>
+    <maxVel>0.1</maxVel>
+  </gazebo>
 </robot>

File: src/arm/urdf_viewer/urdf/robot.urdf (robot description, URDF)
Before this commit: robot urdf, 18 links, 17 joints
Links:
- link part_1: mass 1e-09 -> 0.05
- link part_1_2: mass 1e-09 -> 0.05
- link part_1__length_0_5_meter: mass 1e-09 -> 1.5
Joints:
- joint claw: limit lower=-0.785398 upper=0.279253 effort=10 velocity=10 -> lower=-0.785398 upper=0.279253 effort=20 velocity=10
- joint elbow_1: limit lower=-3.141592653589793 upper=3.141592653589793 effort=10 velocity=10 -> lower=-3.141592653589793 upper=3.141592653589793 effort=30 velocity=10
- joint elbow_2: limit lower=-3.141592653589793 upper=3.141592653589793 effort=10 velocity=10 -> lower=-3.141592653589793 upper=3.141592653589793 effort=30 velocity=10
- joint elbow_end_1: limit lower=-3.141592653589793 upper=3.141592653589793 effort=10 velocity=10 -> lower=-3.141592653589793 upper=3.141592653589793 effort=30 velocity=10
- joint shoulder_1: limit lower=-3.141592653589793 upper=3.141592653589793 effort=10 velocity=10 -> lower=-3.141592653589793 upper=3.141592653589793 effort=50 velocity=10
- joint shoulder_2: limit lower=-3.141592653589793 upper=3.141592653589793 effort=10 velocity=10 -> lower=-3.141592653589793 upper=3.141592653589793 effort=50 velocity=10
- joint shoulder_end_1: limit lower=-3.141592653589793 upper=3.141592653589793 effort=10 velocity=10 -> lower=-3.141592653589793 upper=3.141592653589793 effort=50 velocity=10
- joint slider: limit lower=-0.205617 upper=0.0443825 effort=10 velocity=10 -> lower=-0.205617 upper=0.0443825 effort=50 velocity=10
- joint wrist: limit lower=-3.141592653589793 upper=3.141592653589793 effort=10 velocity=10 -> lower=-3.141592653589793 upper=3.141592653589793 effort=20 velocity=10
